Commit message: renamed the package and respective files for the path

File: urdf/measure_1.urdf (robot description, URDF)
Before this commit: robot measure_1, 2 links, 1 joints
Links:
- link measure_1: geometry collision mesh filename=package://object_anomaly_detection/meshes/measure_1_.STL; visual mesh filename=package://object_anomaly_detection/meshes/measure_1_.STL

File: urdf/measure_2.urdf (robot description, URDF)
Before this commit: robot measure_2, 2 links, 1 joints
Links:
- link measure_2: geometry collision mesh filename=package://object_anomaly_detection/meshes/measure_2_.STL; visual mesh filename=package://object_anomaly_detection/meshes/measure_2_.STL

File: urdf/measure_3.urdf (robot description, URDF)
Before this commit: robot measure_3, 2 links, 1 joints
Links:
- link measure_3: geometry collision mesh filename=package://object_anomaly_detection/meshes/measure_3_.STL; visual mesh filename=package://object_anomaly_detection/meshes/measure_3_.STL

File: urdf/measure_4.urdf (robot description, URDF)
Before this commit: robot measure_4, 2 links, 1 joints
Links:
- link measure_4: geometry collision mesh filename=package://object_anomaly_detection/meshes/measure_4_.STL; visual mesh filename=package://object_anomaly_detection/meshes/measure_4_.STL

File: urdf/robot_rest.urdf (robot description, URDF)
Before this commit: robot robot_rest, 1 links, 0 joints
Links:
- link robot_rest: geometry collision mesh filename=package://object_anomaly_detection/meshes/robot_rest.STL; visual mesh filename=package://object_anomaly_detection/meshes/robot_rest.STL

File: urdf/table.urdf (robot description, URDF)
Before this commit: robot table, 1 links, 0 joints
Links:
- link table: geometry collision mesh filename=package://object_anomaly_detection/meshes/table.STL; visual mesh filename=package://object_anomaly_detection/meshes/table.STL
